Commit message: updated urdf/my_robot.xacro

File: urdf/my_robot.xacro (robot description, xacro)
@@ -1,57 +1,206 @@
 <?xml version='1.0'?>
 <robot name="my_robot" xmlns:xacro="http://www.ros.org/wiki/xacro">
-  <link name="robot_footprint"></link>
-  <joint name="robot_footprint_joint" type="fixed">
-    <origin xyz="0 0 0" rpy="0 0 0" />
-    <parent link="robot_footprint"/>
-    <child link="chassis" />
-  </joint>
-  <link name='chassis'>
-    <pose>0 0 0.1 0 0 0</pose>
-    <inertial>
-      <mass value="15.0"/>
-      <origin xyz="0.0 0 0" rpy=" 0 0 0"/>
-      <inertia
-          ixx="0.1" ixy="0" ixz="0"
-          iyy="0.1" iyz="0"
-          izz="0.1"
-      />
-    </inertial>
-    <collision name='collision'>
-      <origin xyz="0 0 0" rpy=" 0 0 0"/>
-      <geometry>
-        <box size=".4 .2 .1"/>
-      </geometry>
-    </collision>
-    <visual name='chassis_visual'>
-      <origin xyz="0 0 0" rpy=" 0 0 0"/>
-      <geometry>
-        <box size=".4 .2 .1"/>
-      </geometry>
-    </visual>
-    <collision name='back_caster_collision'>
-      <origin xyz="-0.15 0 -0.05" rpy=" 0 0 0"/>
-      <geometry>
-        <sphere radius="0.0499"/>
-      </geometry>
-    </collision>
-    <visual name='back_caster_visual'>
-      <origin xyz="-0.15 0 -0.05" rpy=" 0 0 0"/>
-      <geometry>
-        <sphere radius="0.05"/>
-      </geometry>
-    </visual>
-    <collision name='front_caster_collision'>
-      <origin xyz="0.15 0 -0.05" rpy=" 0 0 0"/>
-      <geometry>
-        <sphere radius="0.0499"/>
-      </geometry>
-    </collision>
-    <visual name='front_caster_visual'>
-      <origin xyz="0.15 0 -0.05" rpy=" 0 0 0"/>
-      <geometry>
-        <sphere radius="0.05"/>
-      </geometry>
-    </visual>
-  </link>
+    <material name="red">
+        <color rgba="0.8 0 0 1"/>
+    </material>
+    <material name="green">
+        <color rgba="0 0.8 0 1"/>
+    </material>
+    <material name="blue">
+        <color rgba="0 0 0.8 1"/>
+    </material>
+    <link name="robot_footprint"></link>
+    <joint name="robot_footprint_joint" type="fixed">
+        <origin xyz="0 0 0" rpy="0 0 0" />
+        <parent link="robot_footprint"/>
+        <child link="chassis" />
+    </joint>
+    <link name='chassis'>
+        <pose>0 0 0.1 0 0 0</pose>
+        <inertial>
+            <mass value="15.0"/>
+            <origin xyz="0.0 0 0" rpy=" 0 0 0"/>
+            <inertia
+                ixx="0.1" ixy="0" ixz="0"
+                iyy="0.1" iyz="0"
+                izz="0.1"
+            />
+        </inertial>
+        <collision name='collision'>
+            <origin xyz="0 0 0" rpy=" 0 0 0"/>
+            <geometry>
+                <box size=".4 .2 .1"/>
+            </geometry>
+        </collision>
+        <visual name='chassis_visual'>
+            <origin xyz="0 0 0" rpy=" 0 0 0"/>
+            <geometry>
+                <box size=".4 .2 .1"/>
+            </geometry>
+            <material name="blue"/>
+        </visual>
+        <collision name='back_caster_collision'>
+            <origin xyz="-0.15 0 -0.05" rpy=" 0 0 0"/>
+            <geometry>
+                <sphere radius="0.0499"/>
+            </geometry>
+        </collision>
+        <visual name='back_caster_visual'>
+            <origin xyz="-0.15 0 -0.05" rpy=" 0 0 0"/>
+            <geometry>
+                <sphere radius="0.05"/>
+            </geometry>
+        </visual>
+        <collision name='front_caster_collision'>
+            <origin xyz="0.15 0 -0.05" rpy=" 0 0 0"/>
+            <geometry>
+                <sphere radius="0.0499"/>
+            </geometry>
+        </collision>
+        <visual name='front_caster_visual'>
+            <origin xyz="0.15 0 -0.05" rpy=" 0 0 0"/>
+            <geometry>
+                <sphere radius="0.05"/>
+            </geometry>
+        </visual>
+    </link>
+    <!-- link for left_wheel -->
+    <link name="left_wheel">
+        <inertial>
+            <mass value="5.0"/>
+            <origin xyz="0.0 0 0" rpy=" 0 0 0"/>
+            <inertia
+                ixx="0.1" ixy="0" ixz="0"
+                iyy="0.1" iyz="0"
+                izz="0.1"
+            />
+        </inertial>
+        <collision>
+            <origin xyz="0 0 0" rpy="0 1.5707 1.5707"/>
+            <geometry>
+                <cylinder radius="0.1" length="0.05" />
+            </geometry>
+        </collision>
+        <visual>
+            <origin xyz="0 0 0" rpy="0 1.5707 1.5707"/>
+            <geometry>
+                <cylinder radius="0.1" length="0.05" />
+            </geometry>
+            <material name="green"/>
+        </visual>
+    </link>
+    <joint type="continuous" name="left_wheel_hinge">
+        <origin xyz="0 0.15 0" rpy="0 0 0"/>
+        <child link="left_wheel"/>
+        <parent link="chassis"/>
+        <axis xyz="0 1 0" rpy="0 0 0"/>
+        <limit effort="10000" velocity="1000"/>
+        <dynamics damping="1.0" friction="1.0"/>
+    </joint>
+    <!-- link for right wheel-->
+    <link name="right_wheel">
+        <inertial>
+            <mass value="5.0"/>
+            <origin xyz="0.0 0 0" rpy=" 0 0 0"/>
+            <inertia
+                ixx="0.1" ixy="0" ixz="0"
+                iyy="0.1" iyz="0"
+                izz="0.1"
+            />
+        </inertial>
+        <collision>
+            <origin xyz="0 0 0" rpy="0 1.5707 1.5707"/>
+            <geometry>
+                <cylinder radius="0.1" length="0.05" />
+            </geometry>
+        </collision>
+        <visual>
+            <origin xyz="0 0 0" rpy="0 1.5707 1.5707"/>
+            <geometry>
+                <cylinder radius="0.1" length="0.05" />
+            </geometry>
+            <material name="green"/>
+        </visual>
+    </link>
+    <joint type="continuous" name="right_wheel_hinge">
+        <origin xyz="0 -0.15 0" rpy="0 0 0"/>
+        <child link="right_wheel"/>
+        <parent link="chassis"/>
+        <axis xyz="0 1 0" rpy="0 0 0"/>
+        <limit effort="10000" velocity="1000"/>
+        <dynamics damping="1.0" friction="1.0"/>
+    </joint>
+    <!-- Camera-->
+    <link name="camera">
+        <inertial>
+            <mass value="0.1"/>
+            <origin xyz="0.05 0.05 0.05" rpy="0 0 0"/>
+            <inertia
+                ixx="1e-6" ixy="0" ixz="0"
+                iyy="1e-6" iyz="0"
+                izz="1e-6"
+            />
+        </inertial>
+        <collision>
+            <origin xyz="0 0 0" rpy="0 0 0"/>
+            <geometry>
+                <box size="0.05 0.05 0.05"/>
+            </geometry>
+        </collision>
+        <visual>
+            <origin xyz="0 0 0" rpy="0 0 0"/>
+            <geometry>
+                <box size="0.05 0.05 0.05"/>
+            </geometry>
+            <material name="red"/>
+        </visual>
+    </link>
+    <joint name="camera_joint" type="fixed">
+        <parent link="chassis"/>
+        <child link="camera"/>
+        <origin xyz="0.2 0 0" rpy="0 0 0"/>
+        <axis value="0 1 0"/>
+    </joint>
+    <!-- lidar-->
+    <link name="hokuyo">
+        <inertial>
+            <mass value="1e-5"/>
+            <origin xyz="0.0 0 0" rpy=" 0 0 0"/>
+            <inertia
+                ixx="1e-6" ixy="0" ixz="0"
+                iyy="1e-6" iyz="0"
+                izz="1e-6"
+            />
+        </inertial>
+        <collision>
+            <origin xyz="0 0 0" rpy="0 0 0"/>
+            <geometry>
+                <box size="0.1 0.1 0.1"/>
+            </geometry>
+        </collision>
+        <visual>
+            <origin xyz="0 0 0" rpy="0 0 0"/>
+            <geometry>
+                <mesh filename="package://my_robot/meshes/hokuyo.dae"/>
+            </geometry>
+        </visual>
+    </link>
+    <joint name="hokuyo_joint" type="fixed">
+        <parent link="chassis"/>
+        <child link="hokuyo"/>
+        <origin xyz="0.15 0 0.1" rpy="0 0 0"/>
+        <axis value="0 1 0"/>
+    </joint>
+    <gazebo reference="left_wheel">
+        <material>Gazebo/Green</material>
+    </gazebo>
+    <gazebo reference="right_wheel">
+        <material>Gazebo/Green</material>
+    </gazebo>
+    <gazebo reference="chassis">
+        <material>Gazebo/Blue</material>
+    </gazebo>
+    <gazebo reference="camera">
+        <material>Gazebo/Red</material>
+    </gazebo>
 </robot>

Commit message: updated urdf/my_robot.xacro imported plugins

File: urdf/my_robot.xacro (robot description, xacro)
@@ -1,4 +1,5 @@
 <?xml version='1.0'?>
 <robot name="my_robot" xmlns:xacro="http://www.ros.org/wiki/xacro">
+	<xacro:include filename="$(find my_robot)/urdf/my_robot.gazebo" />
     <material name="red">
         <color rgba="0.8 0 0 1"/>
@@ -90,5 +91,5 @@
         </visual>
     </link>
-    <joint type="continuous" name="left_wheel_hinge">
+    <joint type="continuous" name="left_wheel_joint">
         <origin xyz="0 0.15 0" rpy="0 0 0"/>
         <child link="left_wheel"/>
@@ -123,5 +124,5 @@
         </visual>
     </link>
-    <joint type="continuous" name="right_wheel_hinge">
+    <joint type="continuous" name="right_wheel_joint">
         <origin xyz="0 -0.15 0" rpy="0 0 0"/>
         <child link="right_wheel"/>

Commit message: updated urdf/my_robot.xacro changed the name of joints

File: urdf/my_robot.xacro (robot description, xacro)
@@ -91,5 +91,5 @@
         </visual>
     </link>
-    <joint type="continuous" name="left_wheel_joint">
+    <joint type="continuous" name="left_wheel_hinge">
         <origin xyz="0 0.15 0" rpy="0 0 0"/>
         <child link="left_wheel"/>
@@ -124,5 +124,5 @@
         </visual>
     </link>
-    <joint type="continuous" name="right_wheel_joint">
+    <joint type="continuous" name="right_wheel_hinge">
         <origin xyz="0 -0.15 0" rpy="0 0 0"/>
         <child link="right_wheel"/>

Commit message: modfied to launch jun.world

File: urdf/my_robot.xacro (robot description, xacro)
@@ -194,14 +194,14 @@
     </joint>
     <gazebo reference="left_wheel">
-        <material>Gazebo/Green</material>
+        <material>Gazebo/Black</material>
     </gazebo>
     <gazebo reference="right_wheel">
-        <material>Gazebo/Green</material>
+        <material>Gazebo/Black</material>
     </gazebo>
     <gazebo reference="chassis">
+        <material>Gazebo/Orange</material>
+    </gazebo>
+    <gazebo reference="camera">
         <material>Gazebo/Blue</material>
     </gazebo>
-    <gazebo reference="camera">
-        <material>Gazebo/Red</material>
-    </gazebo>
 </robot>
